Commit message: a

File: src/simple2wheeler/urdf/simple2wheeler.xacro (robot description, xacro)
@@ -3,8 +3,8 @@
     <link name="link_chassis">
         <pose>0 0 0.1 0 0 0</pose>
-        <inertial>
+      <inertial>
             <mass value="5"/>
             <origin rpy="0 0 0" xyz="0 0 0.1"/>
-            <inertia ixx="0.0395" ixy="0" iyy="0.1062" iyz="0.1062" izz="0.1062"/>
+            <inertia ixx="0.0395" ixy="0" ixz="0"  iyy="0.1062" iyz="0.1062" izz="0.1062"/><!-- -->
         </inertial>
         <collision name="collision_chassis">
@@ -18,4 +18,96 @@
             </geometry>
         </visual>
+        <collision name="caster_front_collision">
+            <origin rpy="0 0 0" xyz="0.20 0 -0.05"/>
+            <geometry>
+                <sphere radius="0.05"/>
+            </geometry>
+            <surface>
+                <friction>
+                    <ode>
+                        <mu>0</mu>
+                        <mu2>0</mu2>
+                        <slip1>1.0</slip1>
+                        <slip2>1.0</slip2>
+                    </ode>
+                </friction>
+            </surface>
+        </collision>
+        <visual name="caster_front_visual">
+            <origin rpy="0 0 0" xyz="0.20 0 -0.05"/>
+            <geometry>
+                <sphere radius="0.05"/>
+            </geometry>
+        </visual>
     </link>
+    <link name="link_right_wheel">
+        <inertial>
+            <mass value="0.2"/>
+            <origin rpy="0 1.57 1.57" xyz="0 0 0"/>
+            <inertia  ixx="0.000526666666667" ixy="0" ixz="0" iyy="0.000526666666667" iyz="0" izz="0.001"/><!-- -->
+        </inertial>
+    <collision name="link_right_wheel_collision">
+        <origin rpy="0 1.5707 1.5707" xyz="0 0 0"/>
+        <geometry>
+            <cylinder length="0.04" radius="0.1"/>
+        </geometry>
+    </collision>
+    <visual name="link_right_wheel_visual">
+        <origin rpy="0 1.5707 1.5707" xyz="0 0 0"/>
+        <geometry>
+            <cylinder length="0.04" radius="0.1"/>
+        </geometry>
+    </visual>
+    </link>
+    <joint name="joint_right_wheel" type="continuous">
+        <origin rpy="0 0 0" xyz="-0.05 0.15 0"/>
+        <child link="link_right_wheel"/>
+        <parent link="link_chassis"/>
+        <axis rpy="0 0 0" xyz="0 1 0"/>
+        <limit effort="1000" velocity="100"/>
+        <joint_properties damping="1.0" friction="1.0"/>
+  </joint>
+      <link name="link_left_wheel">
+        <inertial>
+            <mass value="0.2"/>
+            <origin rpy="0 1.57 1.57" xyz="0 0 0"/>
+            <inertia  ixx="0.000526666666667" ixy="0" ixz="0" iyy="0.000526666666667" iyz="0" izz="0.001"/><!-- -->
+        </inertial>
+    <collision name="link_left_wheel_collision">
+        <origin rpy="0 1.5707 1.5707" xyz="0 0 0"/>
+        <geometry>
+            <cylinder length="0.04" radius="0.1"/>
+        </geometry>
+    </collision>
+    <visual name="link_left_wheel_visual">
+        <origin rpy="0 1.5707 1.5707" xyz="0 0 0"/>
+        <geometry>
+            <cylinder length="0.04" radius="0.1"/>
+        </geometry>
+    </visual>
+    </link>
+    <joint name="joint_left_wheel" type="continuous">
+        <origin rpy="0 0 0" xyz="-0.05 -0.15 0"/>
+        <child link="link_left_wheel"/>
+        <parent link="link_chassis"/>
+        <axis rpy="0 0 0" xyz="0 1 0"/>
+        <limit effort="1000" velocity="100"/>
+        <joint_properties damping="1.0" friction="1.0"/>
+    </joint>
+    <gazebo>
+        <plugin filename="libgazebo_ros_diff_drive.so" name="differential_drive_controller">
+            <legacyMode>false</legacyMode>
+            <alwaysOn>true</alwaysOn>
+            <updateRate>20</updateRate>
+            <leftJoint>joint_left_wheel</leftJoint>
+            <rightJoint>joint_right_wheel</rightJoint>
+            <wheelSeparation>0.2</wheelSeparation>
+            <wheelDiameter>0.2</wheelDiameter>
+            <torque>0.1</torque>
+            <commandTopic>cmd_vel</commandTopic>
+            <odometryTopic>odom</odometryTopic>
+            <odometryFrame>odom</odometryFrame>
+            <robotBaseFrame>link_chassis</robotBaseFrame>
+        </plugin>
+    </gazebo>
 </robot>

Commit message: a

File: src/simple2wheeler/urdf/simple2wheeler.xacro (robot description, xacro)
@@ -95,4 +95,77 @@
         <joint_properties damping="1.0" friction="1.0"/>
     </joint>
+    <link name="camera_link">
+        <collision>
+        </collision>
+        <visual>
+        </visual>
+    </link>
+    <joint name="camera_joint" type="fixed">
+        <origin rpy="0 0 0" xyz="0.25 0.07 0.07"/>
+        <child link="camera_link"/>
+        <parent link="link_chassis"/>
+    </joint>
+    <gazebo reference="camera_link">
+        <sensor type="camera" name="camera_sensor">
+            <update_rate>30</update_rate>
+            <camera>
+                <horizontal_fov>1.3962634</horizontal_fov>
+                <image>
+                    <format>R8G8B8</format>
+                    <width>800</width>
+                    <height>800</height>
+                </image>
+                <clip>
+                    <near>0.01</near>
+                    <far>30</far>
+                </clip>
+            </camera>
+            <plugin name="camera_controller" filename="libgazebo_ros_camera.so">
+                <alwaysOn>true</alwaysOn>
+                <updateRate>30</updateRate>
+                <cameraName>/camera</cameraName>
+                <imageTopicName>image_raw</imageTopicName>
+                <cameraInfoTopicName>camera_info</cameraInfoTopicName>
+                <frameName>camera_link</frameName>
+                <hackBaseline>0.07</hackBaseline>
+                <distortionK1>0.0</distortionK1>
+                <distortionK2>0.0</distortionK2>
+                <distortionK3>0.0</distortionK3>
+                <distortionT1>0.0</distortionT1>
+                <distortionT2>0.0</distortionT2>
+            </plugin>
+        </sensor>
+    </gazebo>
+    <link name="imu_link">
+        <collision>
+        </collision>
+        <visual>
+        </visual>
+    </link>
+    <joint name="imu_joint" type="fixed">
+        <origin rpy="0 0 0" xyz="0 0 0.07"/>
+        <child link="imu_link"/>
+        <parent link="link_chassis"/>
+    </joint>
+    <gazebo reference="imu_link">
+        <gravity>true</gravity>
+        <sensor name="imu_sensor" type="imu">
+            <alwaysOn>true</alwaysOn>
+            <update_rate>10</update_rate>
+            <visualize>true</visualize>
+            <topic>__default_topic__</topic>
+            <plugin filename="libgazebo_ros_imu_sensor.so" name="imu_plugin">
+                <topicName>imu</topicName>
+                <bodyName>imu_link</bodyName>
+                <updateRateHZ>10.0</updateRateHZ>
+                <gaussianNoise>0.0</gaussianNoise>
+                <xyzOffset>0 0 0</xyzOffset>
+                <rpyOffset>0 0 0</rpyOffset>
+                <frameName>imu_link</frameName>
+                <initialOrientationAsReference>false</initialOrientationAsReference>
+            </plugin>
+            <pose>0 0 0 0 0 0</pose>
+        </sensor>
+    </gazebo>
     <gazebo>
         <plugin filename="libgazebo_ros_diff_drive.so" name="differential_drive_controller">
@@ -111,3 +184,57 @@
         </plugin>
     </gazebo>
+    <link name="lidar_link">
+        <visual>
+            <geometry>
+                <mesh filename="package://simple2wheeler/meshes/rplidar_a2_simple.stl" />
+            </geometry>
+        </visual>
+        <collision>
+            <geometry>
+                <mesh filename="package://simple2wheeler/meshes/rplidar_a2_simple.stl" />
+            </geometry>
+        </collision>
+        <inertial>
+            <mass value="0.125"/>
+            <origin zyx="0 0 -0.026"/>
+            <inertia ixx="0.00144185" ixy="0.0" ixz="0.0"
+                    iyy="0.00144185" iyz="0"
+                    izz="0.00144185"/>
+        </inertial>
+    </link>
+    <joint name="lidar_joint" type="fixed">
+        <parent link="link_chassis"/>
+        <child link="lidar_link"/>
+        <origin rpy="0 0 0" xyz="0 0 0.07"/>
+    </joint>
+    <gazebo reference="lidar_link">
+        <sensor type="ray" name="lidar">
+            <alwaysOn>true</alwaysOn>
+            <update_rate>10</update_rate>
+            <pose>0 0 0 0 0 0</pose>
+            <visualize>true</visualize>
+            <ray>
+                <scan>
+                    <horizontal>
+                        <samples>400</samples>
+                        <resolution>0.9</resolution>
+                        <min_angle>-3.142</min_angle>
+                        <max_angle>3.142</max_angle>
+                    </horizontal>
+                </scan>
+                <range>
+                    <min>0.15</min>
+                    <max>6</max>
+                    <resolution>0.01</resolution>
+                </range>
+            </ray>
+            <plugin name="gazebo_ros_lidar_controller" filename="libgazebo_ros_laser.so">
+                <gaussianNoise>0.005</gaussianNoise>
+                <alwaysOn>true</alwaysOn>
+                <updateRate>10</updateRate>
+                <topicName>/lidar</topicName>
+                <frameName>lidar_link</frameName>
+            </plugin>
+        </sensor>
+    </gazebo>
 </robot>
